File: LEOPAD.brd (EAGLE design)
At the start: 74 x 110 mm, 47 parts, among them IC1 ATMEGA32U4-QFN

Commit message: Final tweaks for v1.0 release
Routing:
- net GND: track 39.6 -> 40.6 mm, vias 8 -> 4
Changed lines of the file:
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@@
 <drawing>
 <settings>
-<setting alwaysvectorfont="yes"/>
+<setting alwaysvectorfont="no"/>
 <setting keepoldvectorfont="yes"/>
 <setting verticaltext="up"/>
@@
 <grid distance="1" unitdist="mm" unit="mm" style="dots" multiple="1" display="yes" altdistance="0.001" altunitdist="inch" altunit="inch"/>
 <layers>
-<layer number="1" name="Top" color="4" fill="1" visible="no" active="yes"/>
+<layer number="1" name="Top" color="4" fill="1" visible="yes" active="yes"/>
 <layer number="2" name="Route2" color="1" fill="3" visible="no" active="no"/>
 <layer number="3" name="Route3" color="4" fill="3" visible="no" active="no"/>
@@
 <layer number="14" name="Route14" color="1" fill="6" visible="no" active="no"/>
 <layer number="15" name="Route15" color="4" fill="6" visible="no" active="no"/>
-<layer number="16" name="Bottom" color="1" fill="1" visible="no" active="yes"/>
-<layer number="17" name="Pads" color="2" fill="1" visible="no" active="yes"/>
-<layer number="18" name="Vias" color="2" fill="1" visible="no" active="yes"/>
+<layer number="16" name="Bottom" color="1" fill="1" visible="yes" active="yes"/>
+<layer number="17" name="Pads" color="2" fill="1" visible="yes" active="yes"/>
+<layer number="18" name="Vias" color="2" fill="1" visible="yes" active="yes"/>
 <layer number="19" name="Unrouted" color="6" fill="1" visible="yes" active="yes"/>
 <layer number="20" name="Dimension" color="15" fill="1" visible="yes" active="yes"/>
@@
 <contactref element="XTL1" pad="2"/>
 <contactref element="IC1" pad="TGND"/>
-<via x="39.5" y="94" extent="1-16" drill="0.25" diameter="0.5"/>
+<via x="39.5" y="94" extent="1-16" drill="0.5" diameter="0.5"/>
 <polygon width="0.4064" layer="16">
 <vertex x="0" y="107" curve="-90"/>
@@
 <wire x1="49.6" y1="96" x2="52" y2="96" width="0.254" layer="1"/>
 <wire x1="52" y1="96" x2="53" y2="95" width="0.254" layer="1"/>
-<wire x1="56.4" y1="97" x2="55" y2="97" width="0.254" layer="1"/>
-<wire x1="55" y1="97" x2="53.5" y2="97" width="0.254" layer="1"/>
+<wire x1="56.4" y1="97" x2="53.5" y2="97" width="0.254" layer="1"/>
 <wire x1="50.5" y1="91.6" x2="50.5" y2="93.5" width="0.254" layer="1"/>
 <wire x1="52" y1="95" x2="53" y2="95" width="0.254" layer="1"/>
@@
 <wire x1="56.4" y1="97" x2="58" y2="97" width="0.254" layer="1"/>
 <wire x1="56.4" y1="93" x2="58" y2="93" width="0.254" layer="1"/>
-<via x="55" y="93" extent="1-16" drill="0.5"/>
-<via x="55" y="97" extent="1-16" drill="0.5"/>
-<via x="51" y="97" extent="1-16" drill="0.5"/>
-<via x="51" y="93" extent="1-16" drill="0.5"/>
 <wire x1="42.5" y1="93.238" x2="40.788" y2="93.238" width="0.254" layer="1"/>
 <wire x1="40.788" y1="93.238" x2="40.65" y2="93.1" width="0.254" layer="1"/>
-<wire x1="49.6" y1="96" x2="48" y2="96" width="0.254" layer="1"/>
+<wire x1="49.6" y1="96" x2="47" y2="96" width="0.254" layer="1"/>
 <via x="56.7" y="99" extent="1-16" drill="0.5"/>
 <via x="55.4" y="101" extent="1-16" drill="0.5"/>
@@
 <contactref element="IC1" pad="9"/>
 <contactref element="ICSP" pad="3"/>
-<wire x1="54.5996625" y1="103" x2="52" y2="103" width="0.254" layer="16"/>
+<wire x1="52" y1="103" x2="54.5996625" y2="103" width="0.254" layer="16"/>
 <wire x1="52" y1="103" x2="51" y2="102" width="0.254" layer="16"/>
 <wire x1="51" y1="102" x2="51" y2="100" width="0.254" layer="16"/>
@@
 <wire x1="51.5" y1="98.4" x2="51.5" y2="99.5" width="0.254" layer="1"/>
 <wire x1="51.5" y1="99.5" x2="51" y2="100" width="0.254" layer="1"/>
-<wire x1="62.37" y1="95.2964" x2="61.6842" y2="95.9822" width="0.254" layer="16"/>
-<wire x1="61.6842" y1="95.9822" x2="61.6174625" y2="95.9822" width="0.254" layer="16"/>
-<wire x1="61.6174625" y1="95.9822" x2="54.5996625" y2="103" width="0.254" layer="16"/>
+<wire x1="62.3032625" y1="95.2964" x2="62.37" y2="95.2964" width="0.254" layer="16"/>
+<wire x1="54.5996625" y1="103" x2="62.3032625" y2="95.2964" width="0.254" layer="16"/>
 </signal>
 <signal name="MOSI">
@@
 <wire x1="50" y1="100" x2="50" y2="102" width="0.254" layer="16"/>
 <wire x1="50" y1="102" x2="52" y2="104" width="0.254" layer="16"/>
-<wire x1="52" y1="104" x2="54.1744" y2="104" width="0.254" layer="16"/>
 <wire x1="63.91460625" y1="95.2964" x2="64.91" y2="95.2964" width="0.254" layer="16"/>
-<wire x1="61.7858" y1="96.3886" x2="62.82240625" y2="96.3886" width="0.254" layer="16"/>
 <wire x1="62.82240625" y1="96.3886" x2="63.91460625" y2="95.2964" width="0.254" layer="16"/>
-<wire x1="54.1744" y1="104" x2="61.7858" y2="96.3886" width="0.254" layer="16"/>
+<wire x1="61.2778" y1="97.7222" x2="61.2778" y2="97.38399375" width="0.254" layer="16"/>
+<wire x1="61.2778" y1="97.38399375" x2="62.27319375" y2="96.3886" width="0.254" layer="16"/>
+<wire x1="62.27319375" y1="96.3886" x2="62.82240625" y2="96.3886" width="0.254" layer="16"/>
+<wire x1="55" y1="104" x2="61.2778" y2="97.7222" width="0.254" layer="16"/>
+<wire x1="52" y1="104" x2="55" y2="104" width="0.254" layer="16"/>
 </signal>
 <signal name="MISO">
@@
 <wire x1="54.5" y1="91.6" x2="54.5" y2="90.5" width="0.254" layer="1"/>
 <wire x1="56" y1="89" x2="64" y2="89" width="0.254" layer="1"/>
-<via x="64" y="89" extent="1-16" drill="0.35"/>
+<via x="64" y="89" extent="1-16" drill="0.5"/>
 <wire x1="64" y1="89" x2="63" y2="88" width="0.254" layer="16"/>
 <wire x1="63" y1="88" x2="53" y2="88" width="0.254" layer="16"/>
@@
 <wire x1="38" y1="99.5" x2="37.75" y2="99.75" width="0.2032" layer="1"/>
 <wire x1="40" y1="99.5" x2="38" y2="99.5" width="0.254" layer="1"/>
-<wire x1="37.75" y1="99.75" x2="37.75" y2="101.44" width="0.2032" layer="1"/>
+<wire x1="37.75" y1="99.75" x2="37.75" y2="100.11895" width="0.2032" layer="1"/>
+<wire x1="37.75" y1="100.11895" x2="37.6952" y2="100.17375" width="0.2032" layer="1"/>
+<wire x1="37.6952" y1="100.17375" x2="37.6952" y2="100.72625" width="0.2032" layer="1"/>
+<wire x1="37.6952" y1="100.72625" x2="37.75" y2="100.78105" width="0.2032" layer="1"/>
+<wire x1="37.75" y1="100.78105" x2="37.75" y2="101.44" width="0.2032" layer="1"/>
 </signal>
 <signal name="A4">
@@
 </signal>
 </signals>
+<errors>
+</errors>
 </board>
 </drawing>
